File: bikeLights.kicad_pcb (KiCad board)
At the start: 2 copper layers, 71.1 x 66 mm, 24 parts, among them J1 Battery, J2 Light Sensor, J3 Front Light, J4 Rear Lights, J5 Hub Power In, Q1 IRF9540N, Q2 P2N2222A, Q3 RFP30N06LE, Q4 P2N2222A

Commit message: Updates
Parts:
- moved J4 0.64 mm to (92.7, 92.1)
- moved Q4 0.63 mm to (101.0, 92.1), turned to -90 degrees
Connections:
- D1 pad 1: Net-(C1-Pad1) -> Net-(A1-Pad30)
- D1 pad 2: Net-(A1-Pad30) -> Net-(C1-Pad1)
- J5 pad 1: Net-(D2-Pad2) -> Net-(D2-Pad3)
- J5 pad 2: Net-(D2-Pad3) -> Net-(D2-Pad2)
Routing:
- net GND: track 12.4 -> 1.22 mm
- net Net-(Q1-Pad2): track 36.9 -> 28.4 mm, vias 2 -> 0
- net Net-(A1-Pad27): track 49.0 -> 45.0 mm
- net Net-(Q4-Pad2): track 11.0 -> 13.3 mm
- net Net-(A1-Pad20): track 35.3 -> 33.9 mm, vias 2 -> 1
- net Net-(J4-Pad2): track 9.20 -> 8.27 mm
- net Net-(A1-Pad5): vias 4 -> 2
Other:
- board text added: "+ -"
- board text added: "Bike Lights Board V1 2-27-23"

Commit message: updates
Parts:
- J1, J2, J3, J4, J5: footprint Connector_Wire:SolderWire-0.1sqmm_1x02_P3.6mm_D0.4mm_OD1mm -> solder_pads:solder_pads_medium
- moved J5 2.76 mm to (93.2, 126.8), turned to -90 degrees
- moved J3 1.91 mm to (93.3, 77.5)
- moved J1 1.42 mm to (158.1, 88.9)
- moved J2 1.42 mm to (93.3, 109.2)
- moved J4 1.42 mm to (93.3, 93.3)
- moved D2 0.81 mm to (104.7, 132.8)
- moved Q4 0.51 mm to (101.0, 92.6), turned to 90 degrees
- turned Q2 to 180 degrees
Connections:
- Q2 pad 1: Net-(Q2-Pad1) -> GND
- Q2 pad 3: GND -> Net-(Q2-Pad3)
- Q4 pad 1: Net-(J4-Pad2) -> GND
- Q4 pad 3: GND -> Net-(J4-Pad2)
- R4 pad 2: Net-(Q2-Pad1) -> Net-(Q2-Pad3)
Routing:
- net Net-(Q2-Pad1): track 12.2 -> 0.00 mm
- net Net-(Q2-Pad3): track 0.00 -> 11.8 mm
- net Net-(A1-Pad30): track 132.8 -> 126.2 mm
- net Net-(Q4-Pad2): track 13.3 -> 10.1 mm
- net Net-(Q2-Pad2): track 18.6 -> 20.1 mm
- net GND: track 1.22 -> 0.00 mm
- net Net-(C1-Pad1): track 71.0 -> 70.2 mm
- net Net-(A1-Pad19): track 54.4 -> 53.6 mm
- net Net-(J4-Pad2): track 8.27 -> 7.51 mm
- net Net-(J3-Pad2): track 30.0 -> 29.2 mm
- net Net-(D2-Pad3): track 12.2 -> 11.6 mm
Other:
- board size 71.1 x 66 mm -> 70.5 x 64.1 mm

Commit message: Updates
Parts:
- J1, J2, J5: footprint solder_pads:solder_pads_medium -> solder_pads:solder_holes_medium
- J3: value Front Light -> Front Light - +; footprint solder_pads:solder_pads_medium -> solder_pads:solder_holes_medium
- J4: value Rear Lights -> Rear Lights - +; footprint solder_pads:solder_pads_medium -> solder_pads:solder_holes_medium
Routing:
- net Net-(Q1-Pad2): track 28.4 -> 29.6 mm
- net Net-(J1-Pad1): track 37.5 -> 38.3 mm, vias 0 -> 1
- net Net-(D2-Pad2): track 12.1 -> 12.7 mm
Other:
- board size 70.5 x 64.1 mm -> 71.1 x 64.1 mm
