File: bikeLights.kicad_sch (KiCad schematic)
At the start: 24 parts, among them J1 Battery, J2 Light Sensor, J3 Front Light, J4 Rear Lights, J5 Hub Power In, Q1 IRF9540N, Q2 P2N2222A, Q3 RFP30N06LE, Q4 P2N2222A

Commit message: Updates
Connections:
- net at D2.2: now also J5.2 (Pin_2); no longer J5.1 (Pin_1)
- net at D2.3: now also J5.1 (Pin_1); no longer J5.2 (Pin_2)
Other:
- moved on the sheet: J5
Changed lines of the file:
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@@
       (effects (font (size 1.27 1.27)) hide)
     )
+    (pin "1")
     (pin "2")
-    (pin "1")
   )
-  (symbol (lib_id "Connector:Conn_01x02_Male") (at 264.16 36.83 180) (unit 1)
+  (symbol (lib_id "Connector:Conn_01x02_Male") (at 264.16 34.29 0) (mirror y) (unit 1)
     (in_bom yes) (on_board yes)
-    (property "Reference" "J5" (id 0) (at 263.525 41.91 0))
-    (property "Value" "Hub Power In" (id 1) (at 263.525 39.37 0))
-    (property "Footprint" "Connector_Wire:SolderWire-0.1sqmm_1x02_P3.6mm_D0.4mm_OD1mm" (id 2) (at 264.16 36.83 0)
+    (property "Reference" "J5" (id 0) (at 264.16 31.75 0))
+    (property "Value" "Hub Power In" (id 1) (at 264.16 39.37 0))
+    (property "Footprint" "Connector_Wire:SolderWire-0.1sqmm_1x02_P3.6mm_D0.4mm_OD1mm" (id 2) (at 264.16 34.29 0)
       (effects (font (size 1.27 1.27)) hide)
     )
-    (property "Datasheet" "~" (id 3) (at 264.16 36.83 0)
+    (property "Datasheet" "~" (id 3) (at 264.16 34.29 0)
       (effects (font (size 1.27 1.27)) hide)
     )

Commit message: updates
Parts:
- J1, J2, J3, J4, J5: footprint Connector_Wire:SolderWire-0.1sqmm_1x02_P3.6mm_D0.4mm_OD1mm -> solder_pads:solder_pads_medium
Connections:
- net GND: now also Q2.1 (E), Q4.1 (E); no longer Q2.3 (E), Q4.3 (E)
- net at R4.2: now also Q2.3 (C); no longer Q2.1 (C)
- net at J4.2 (Pin_2): now also Q4.3 (C); no longer Q4.1 (C)
Changed lines of the file:
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@@
   (symbol (lib_name "Q_NPN_BCE_1") (lib_id "Device:Q_NPN_BCE") (at 93.98 60.96 0) (mirror y) (unit 1)
     (in_bom yes) (on_board yes) (fields_autoplaced)
-    (property "Reference" "Q2" (id 0) (at 99.06 59.6899 0)
-      (effects (font (size 1.27 1.27)) (justify left))
-    )
-    (property "Value" "P2N2222A" (id 1) (at 99.06 62.23 0)
-      (effects (font (size 1.27 1.27)) (justify left))
-    )
-    (property "Footprint" "eec:ON_Semi-CASE_2911-0-0-0" (id 2) (at 99.06 58.42 0)
+    (property "Reference" "Q2" (id 0) (at 88.9 59.6899 0)
+      (effects (font (size 1.27 1.27)) (justify left))
+    )
+    (property "Value" "P2N2222A" (id 1) (at 88.9 62.23 0)
+      (effects (font (size 1.27 1.27)) (justify left))
+    )
+    (property "Footprint" "eec:ON_Semi-CASE_2911-0-0-0" (id 2) (at 88.9 58.42 0)
       (effects (font (size 1.27 1.27)) hide)
     )
@@
   (symbol (lib_id "Device:Q_NPN_BCE") (at 73.66 100.33 90) (unit 1)
     (in_bom yes) (on_board yes) (fields_autoplaced)
-    (property "Reference" "Q4" (id 0) (at 64.77 100.33 90))
-    (property "Value" "P2N2222A" (id 1) (at 67.31 100.33 90))
-    (property "Footprint" "eec:ON_Semi-CASE_2911-0-0-0" (id 2) (at 68.58 102.87 0)
+    (property "Reference" "Q4" (id 0) (at 73.66 109.22 90))
+    (property "Value" "P2N2222A" (id 1) (at 73.66 106.68 90))
+    (property "Footprint" "eec:ON_Semi-CASE_2911-0-0-0" (id 2) (at 76.2 105.41 0)
       (effects (font (size 1.27 1.27)) hide)
     )
@@
       (effects (font (size 1.27 1.27)) (justify right))
     )
-    (property "Footprint" "Connector_Wire:SolderWire-0.1sqmm_1x02_P3.6mm_D0.4mm_OD1mm" (id 2) (at 54.61 27.94 0)
+    (property "Footprint" "solder_pads:solder_pads_medium" (id 2) (at 54.61 27.94 0)
       (effects (font (size 1.27 1.27)) hide)
     )
@@
     (property "Reference" "J3" (id 0) (at 83.185 124.46 0))
     (property "Value" "Front Light" (id 1) (at 83.185 127 0))
-    (property "Footprint" "Connector_Wire:SolderWire-0.1sqmm_1x02_P3.6mm_D0.4mm_OD1mm" (id 2) (at 82.55 129.54 0)
+    (property "Footprint" "solder_pads:solder_pads_medium" (id 2) (at 82.55 129.54 0)
       (effects (font (size 1.27 1.27)) hide)
     )
@@
     (property "Reference" "J5" (id 0) (at 264.16 31.75 0))
     (property "Value" "Hub Power In" (id 1) (at 264.16 39.37 0))
-    (property "Footprint" "Connector_Wire:SolderWire-0.1sqmm_1x02_P3.6mm_D0.4mm_OD1mm" (id 2) (at 264.16 34.29 0)
+    (property "Footprint" "solder_pads:solder_pads_medium" (id 2) (at 264.16 34.29 0)
       (effects (font (size 1.27 1.27)) hide)
     )
@@
       (effects (font (size 1.27 1.27)) (justify right))
     )
-    (property "Footprint" "Connector_Wire:SolderWire-0.1sqmm_1x02_P3.6mm_D0.4mm_OD1mm" (id 2) (at 242.57 66.04 0)
+    (property "Footprint" "solder_pads:solder_pads_medium" (id 2) (at 242.57 66.04 0)
       (effects (font (size 1.27 1.27)) hide)
     )
@@
     (property "Reference" "J4" (id 0) (at 60.325 90.17 0))
     (property "Value" "Rear Lights" (id 1) (at 59.69 92.71 0))
-    (property "Footprint" "Connector_Wire:SolderWire-0.1sqmm_1x02_P3.6mm_D0.4mm_OD1mm" (id 2) (at 59.69 95.25 0)
+    (property "Footprint" "solder_pads:solder_pads_medium" (id 2) (at 59.69 95.25 0)
       (effects (font (size 1.27 1.27)) hide)
     )
@@
     )
     (path "/6eee0dd2-64a0-4043-8d7e-2423cf8efb4f"
-      (reference "J1") (unit 1) (value "Battery") (footprint "Connector_Wire:SolderWire-0.1sqmm_1x02_P3.6mm_D0.4mm_OD1mm")
+      (reference "J1") (unit 1) (value "Battery") (footprint "solder_pads:solder_pads_medium")
     )
     (path "/b2018b95-c579-460f-aa95-24ba99f6f45e"
-      (reference "J2") (unit 1) (value "Light Sensor") (footprint "Connector_Wire:SolderWire-0.1sqmm_1x02_P3.6mm_D0.4mm_OD1mm")
+      (reference "J2") (unit 1) (value "Light Sensor") (footprint "solder_pads:solder_pads_medium")
     )
     (path "/709ef163-7b76-44f9-9487-8077dba5a51a"
-      (reference "J3") (unit 1) (value "Front Light") (footprint "Connector_Wire:SolderWire-0.1sqmm_1x02_P3.6mm_D0.4mm_OD1mm")
+      (reference "J3") (unit 1) (value "Front Light") (footprint "solder_pads:solder_pads_medium")
     )
     (path "/c163059a-fee3-45ae-a226-449589aaeb85"
-      (reference "J4") (unit 1) (value "Rear Lights") (footprint "Connector_Wire:SolderWire-0.1sqmm_1x02_P3.6mm_D0.4mm_OD1mm")
+      (reference "J4") (unit 1) (value "Rear Lights") (footprint "solder_pads:solder_pads_medium")
     )
     (path "/733b1374-0b54-44dd-927b-832b94d39d76"
-      (reference "J5") (unit 1) (value "Hub Power In") (footprint "Connector_Wire:SolderWire-0.1sqmm_1x02_P3.6mm_D0.4mm_OD1mm")
+      (reference "J5") (unit 1) (value "Hub Power In") (footprint "solder_pads:solder_pads_medium")
     )
     (path "/81e65906-9297-413e-a103-4779d56f2725"

Commit message: Updates
Parts:
- J1, J2, J3, J4, J5: footprint solder_pads:solder_pads_medium -> solder_pads:solder_holes_medium
Changed lines of the file:
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@@
       (effects (font (size 1.27 1.27)) (justify right))
     )
-    (property "Footprint" "solder_pads:solder_pads_medium" (id 2) (at 54.61 27.94 0)
+    (property "Footprint" "solder_pads:solder_holes_medium" (id 2) (at 54.61 27.94 0)
       (effects (font (size 1.27 1.27)) hide)
     )
@@
     (property "Reference" "J3" (id 0) (at 83.185 124.46 0))
     (property "Value" "Front Light" (id 1) (at 83.185 127 0))
-    (property "Footprint" "solder_pads:solder_pads_medium" (id 2) (at 82.55 129.54 0)
+    (property "Footprint" "solder_pads:solder_holes_medium" (id 2) (at 82.55 129.54 0)
       (effects (font (size 1.27 1.27)) hide)
     )
@@
     (property "Reference" "J5" (id 0) (at 264.16 31.75 0))
     (property "Value" "Hub Power In" (id 1) (at 264.16 39.37 0))
-    (property "Footprint" "solder_pads:solder_pads_medium" (id 2) (at 264.16 34.29 0)
+    (property "Footprint" "solder_pads:solder_holes_medium" (id 2) (at 264.16 34.29 0)
       (effects (font (size 1.27 1.27)) hide)
     )
@@
       (effects (font (size 1.27 1.27)) (justify right))
     )
-    (property "Footprint" "solder_pads:solder_pads_medium" (id 2) (at 242.57 66.04 0)
+    (property "Footprint" "solder_pads:solder_holes_medium" (id 2) (at 242.57 66.04 0)
       (effects (font (size 1.27 1.27)) hide)
     )
@@
     (property "Reference" "J4" (id 0) (at 60.325 90.17 0))
     (property "Value" "Rear Lights" (id 1) (at 59.69 92.71 0))
-    (property "Footprint" "solder_pads:solder_pads_medium" (id 2) (at 59.69 95.25 0)
+    (property "Footprint" "solder_pads:solder_holes_medium" (id 2) (at 59.69 95.25 0)
       (effects (font (size 1.27 1.27)) hide)
     )
@@
     )
     (path "/6eee0dd2-64a0-4043-8d7e-2423cf8efb4f"
-      (reference "J1") (unit 1) (value "Battery") (footprint "solder_pads:solder_pads_medium")
+      (reference "J1") (unit 1) (value "Battery") (footprint "solder_pads:solder_holes_medium")
     )
     (path "/b2018b95-c579-460f-aa95-24ba99f6f45e"
-      (reference "J2") (unit 1) (value "Light Sensor") (footprint "solder_pads:solder_pads_medium")
+      (reference "J2") (unit 1) (value "Light Sensor") (footprint "solder_pads:solder_holes_medium")
     )
     (path "/709ef163-7b76-44f9-9487-8077dba5a51a"
-      (reference "J3") (unit 1) (value "Front Light") (footprint "solder_pads:solder_pads_medium")
+      (reference "J3") (unit 1) (value "Front Light") (footprint "solder_pads:solder_holes_medium")
     )
     (path "/c163059a-fee3-45ae-a226-449589aaeb85"
-      (reference "J4") (unit 1) (value "Rear Lights") (footprint "solder_pads:solder_pads_medium")
+      (reference "J4") (unit 1) (value "Rear Lights") (footprint "solder_pads:solder_holes_medium")
     )
     (path "/733b1374-0b54-44dd-927b-832b94d39d76"
-      (reference "J5") (unit 1) (value "Hub Power In") (footprint "solder_pads:solder_pads_medium")
+      (reference "J5") (unit 1) (value "Hub Power In") (footprint "solder_pads:solder_holes_medium")
     )
     (path "/81e65906-9297-413e-a103-4779d56f2725"
